Commit message: modify goal publisher

File: urdf/robot2.urdf (robot description, URDF)
Before this commit: robot one_arm, 7 links, 6 joints
Joints:
- joint pointer_joint: origin xyz=0.02 0 0.03 rpy=0 0.593 0 -> xyz=0.02 0 -0.03 rpy=0 -0.593 0

Commit message: sensing ok

File: urdf/robot2.urdf (robot description, URDF)
Before this commit: robot one_arm, 7 links, 6 joints
Links:
- added link sense_link; visual mesh filename=package://sfp03/urdf/ViveController.stl
- link link1: geometry visual cylinder length=0.1 radius=0.11
- link link2: geometry visual box size=0.06 0.1 0.04
Joints:
- added joint sense_joint: type fixed, parent base_link, child sense_link, origin xyz=0.03 -0.04 0.190 rpy=0 0 0
- joint joint2: origin xyz=0.08 0 0.1 rpy=0 0 0 -> xyz=0.06 0 0.1 rpy=0 0 0
- joint robot_joint: type planar -> floating
