Commit message: sfp3 presentation

File: urdf/robot.urdf (robot description, URDF)
Before this commit: robot one_arm, 6 links, 5 joints
Links:
- removed link link1
- removed link link2
- removed link temp1
- removed link temp2
- removed link world
- link base_link: geometry visual cylinder length=0.10 radius=0.15
Joints:
- removed joint joint1
- removed joint joint2
- removed joint robot_joint1
- removed joint robot_joint2
- removed joint robot_joint3
